File: mycoil/mycoil.kicad_pcb (KiCad board)
At the start: 4 copper layers, 39.2 x 39.2 mm, 0 parts

Commit message: add
Routing:
- net (no net): track 50388.6 -> 0.00 mm, vias 2 -> 0
Other:
- copper layers 4 -> 8

Commit message: readme
Routing:
- net (no net): track 0.00 -> 50628.4 mm, vias 0 -> 5
